File: SunSensorMux.kicad_sch (KiCad schematic)
At the start: 6 parts, among them U1 TCA9548A_Multiplexer

Commit message: Fixed net issues
Parts:
- removed L1, L2, L3, L4, L5: Adafruit_VEML7700_Lux_Sensor, symbol Sensor_Optical:Adafruit_VEML7700_Lux_Sensor
- added J1, J2: Conn_01x03, symbol Connector_Generic:Conn_01x03
- added L1, L2, L3, L4, L5: VEML7700_Lux_Sensor, symbol Sensor_Optical:VEML7700_Lux_Sensor
- U1: footprint (none) -> sunsensor:SOP65P640X120-24N
Connections:
- net at U1.5 (SCL0): now also L1.1 (SCL)
- net at U1.4 (SDA0): now also L1.5 (SDA)
- net at U1.7 (SCL1): now also L3.1 (SCL)
- net at U1.6 (SDA1): now also L3.5 (SDA)
- net at U1.1 (A0): now also J2.1 (Pin_1)
- net at U1.10 (SDA3): now also L2.5 (SDA)
- net at U1.11 (SCL3): now also L2.1 (SCL)
- net GND: now reaches U1.12 (GND)
- net GND: now also U1.15 (SDA5), U1.17 (SDA6), U1.19 (SDA7), U1.20 (SCL7), L1.3 (GND), L2.3 (GND), L3.3 (GND), L4.3 (GND), L5.3 (GND)
- net at U1.13 (SDA4): now also L4.5 (SDA)
- net at U1.14 (SCL4): now also L4.1 (SCL)
- net at U1.2 (A1): now also J2.2 (Pin_2)
- net at U1.21 (A2): now also J2.3 (Pin_3)
- net at U1.22 (SCL): now also J1.2 (Pin_2)
- net at U1.23 (SDA): now also J1.3 (Pin_3)
- net at U1.3 (RESET): now also J1.1 (Pin_1)
- net at U1.8 (SDA2): now also L5.5 (SDA)
- net at U1.9 (SCL2): now also L5.1 (SCL)
- new net +3.3VDAC: L1.2 (Vin), L2.2 (Vin), L3.2 (Vin), L4.2 (Vin), L5.2 (Vin)
