File: SunSensor/SunSensor.kicad_pcb (KiCad board)
At the start: 2 copper layers, 16 parts, among them U1 AD7291BCPZ

Commit message: Finished traces
Parts:
- added U2: FEATHER_M0_BASIC_PROTO, sunsensor:MODULE_FEATHER_M0_BASIC_PROTO, F.Cu at (165.4, 98.4)
- moved AlertLED1 8.25 mm to (132.8, 108.1)
- moved C3 0.45 mm to (129.0, 104.4)
Connections:
- C1 pad 2: GNDS -> GNDREF
- C2 pad 2: GNDS -> GNDREF
- C3 pad 2: GNDS -> GNDREF
- U1 pad 11: unconnected-(U1-Pad11) -> /AS0
- U1 pad 13: unconnected-(U1-Pad13) -> /AS1
- U1 pad 14: unconnected-(U1-Pad14) -> /SDA_chip
- U1 pad 15: unconnected-(U1-Pad15) -> /SCL_chip
- U1 pad 16: unconnected-(U1-Pad16) -> +3V3
- U1 pad 21: (no net) -> GNDREF
Routing:
- net /SDA_chip: track 0.00 -> 65.4 mm, vias 0 -> 2
- net /SCL_chip: track 0.00 -> 62.5 mm, vias 0 -> 2
- net /V_ref: track 0.00 -> 53.8 mm, vias 0 -> 2
- net /AS0: track 0.00 -> 48.1 mm
- net /AS1: track 0.00 -> 46.2 mm
- net GNDS: track 4.72 -> 38.7 mm, vias 0 -> 2
- net /Vin5: track 3.49 -> 26.9 mm, vias 0 -> 2
- net +3V3: track 24.0 -> 44.1 mm
- net /Vin4: track 3.90 -> 18.7 mm, vias 0 -> 2
- net /Vin2: track 3.59 -> 17.6 mm, vias 0 -> 2
- net /Vin1: track 4.45 -> 14.2 mm
- net /Vin3: track 3.99 -> 13.0 mm
- net Net-(AlertLED1-Pad1): track 8.25 -> 13.8 mm, vias 0 -> 2
- net GNDREF: track 26.9 -> 22.8 mm, vias 0 -> 12
- added copper zone on B.Cu, net GNDREF
- added copper zone on B.Cu, net GNDS
Other:
- board outline added: 92.9 x 34.7 mm

Commit message: Final modifications
Parts:
- added C4: 10 µF, sunsensor:CAPC1005X71N, F.Cu at (114.9, 104.8)
Connections:
- AlertLED1 pad 2: (no net) -> /LEDOUT
- R11 pad 1: Net-(AlertLED1-Pad20) -> /LEDOUT
- U1 pad 21: GNDREF -> (no net)
- U2 pad P$1: GNDREF -> (no net)
- U2 pad P$2: GNDREF -> (no net)
Routing:
- net GNDREF: track 22.8 -> 88.3 mm, vias 12 -> 16
- net /LEDOUT: track 0.00 -> 22.1 mm, vias 0 -> 2
- net GNDS: track 38.7 -> 16.7 mm, vias 2 -> 0
- net /V_ref: track 53.8 -> 55.8 mm
- net /Vin3: track 13.0 -> 14.8 mm
- net /Vin2: track 17.6 -> 19.3 mm
- net /Vin4: track 18.7 -> 17.2 mm
- net /Vin5: track 26.9 -> 27.9 mm
- removed copper zone on B.Cu, net GNDS

Commit message: Small fixes
Parts:
- added C5: 10 µF, sunsensor:CAPC1005X71N, F.Cu at (124.6, 97.0)
Connections:
- AlertLED1 pad 2: /LEDOUT -> (no net)
- U1 pad 18: GNDS -> GNDREF
Routing:
- net +3V3: track 44.1 -> 79.1 mm, vias 0 -> 1
- net GNDREF: track 88.3 -> 91.9 mm
- net GNDS: track 16.7 -> 14.8 mm

Commit message: more small changes
Connections:
- AlertLED1 pad 2: (no net) -> /LEDOUT
- C4 pad 2: GNDS -> GNDREF
- U1 pad 21: (no net) -> GNDREF
- U1 pad 4: GNDS -> GNDREF
- U1 pad 5: GNDS -> GNDREF
- U1 pad 6: GNDS -> GNDREF
- U2 pad P$1: (no net) -> GNDREF
- U2 pad P$2: (no net) -> GNDREF
Routing:
- net GNDS: track 14.8 -> 0.00 mm
- net GNDREF: track 91.9 -> 100.1 mm, vias 16 -> 14
- net +3V3: track 79.1 -> 80.5 mm

Commit message: Finish Routing
Parts:
- added R6: 10K, Resistor_SMD:R_0603_1608Metric, F.Cu at (127.3, 99.1)
- added R7: 10K, Resistor_SMD:R_0603_1608Metric, F.Cu at (128.8, 99.1)
- Alert: renamed from AlertLED1; footprint sunsensor:LED_77&slash_TR8_EVE -> LED_SMD:LED_0603_1608Metric
- C1: value 1 µF -> 1uF; footprint sunsensor:CAPC1005X60N -> Capacitor_SMD:C_0603_1608Metric
- C2: value 100 µF -> 10uF; footprint sunsensor:CAPC3216X190N -> Capacitor_SMD:C_0603_1608Metric
- C3: value 100 nF -> 0.1uF; footprint sunsensor:CAPC1005X55N -> Capacitor_SMD:C_0603_1608Metric
- C4: value 10 µF -> 10uF; footprint sunsensor:CAPC1005X71N -> Capacitor_SMD:C_0603_1608Metric
- C5: value 10 µF -> 1uF; footprint sunsensor:CAPC1005X71N -> Capacitor_SMD:C_0603_1608Metric
- R1: renamed from R2; value 50k_Ohms -> 50K; footprint sunsensor:RESC3116X65N -> Resistor_SMD:R_0603_1608Metric
- R2: renamed from R6; value 50k_Ohms -> 50K; footprint sunsensor:RESC3116X65N -> Resistor_SMD:R_0603_1608Metric
- R3: renamed from R10; value 50k_Ohms -> 50K; footprint sunsensor:RESC3116X65N -> Resistor_SMD:R_0603_1608Metric
- R4: value 50k_Ohms -> 50K; footprint sunsensor:RESC3116X65N -> Resistor_SMD:R_0603_1608Metric
- R5: renamed from R8; value 50k_Ohms -> 50K; footprint sunsensor:RESC3116X65N -> Resistor_SMD:R_0603_1608Metric
- R8: renamed from R11; value 1k_ohms -> 1K; footprint sunsensor:RESC3216X75N -> Resistor_SMD:R_0603_1608Metric
- U1: footprint sunsensor:QFN50P400X400X100-21N -> Package_DFN_QFN:QFN-20-1EP_4x4mm_P0.5mm_EP2.6x2.6mm
- U2: footprint sunsensor:MODULE_FEATHER_M0_BASIC_PROTO -> Module:Adafruit_Feather
- moved U2 21.4 mm to (146.2, 107.8), turned to 90 degrees
- moved R8 20.8 mm to (131.2, 102.2), turned to 0 degrees
- moved R3 17.2 mm to (114.0, 90.7)
- moved MOSFET3 16.1 mm to (114.0, 85.7)
- moved R4 10.2 mm to (109.0, 90.7)
- moved MOSFET4 9.77 mm to (109.0, 85.7)
- moved C1 8.60 mm to (122.0, 106.2), turned to -90 degrees
- moved Alert 7.61 mm to (128.0, 102.2), turned to 180 degrees
- moved R2 7.21 mm to (119.0, 90.7)
- moved MOSFET2 7.06 mm to (119.0, 85.7)
- moved C4 5.81 mm to (120.5, 106.2), turned to -90 degrees
- moved C2 5.32 mm to (124.0, 106.2), turned to -90 degrees
- moved C3 3.95 mm to (125.5, 106.2)
- moved R1 3.59 mm to (124.0, 90.7)
- moved R5 2.58 mm to (104.0, 90.7)
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- renumbered MOSFET3 to MOSFET2, MOSFET5 to MOSFET3, MOSFET2 to MOSFET4, MOSFET4 to MOSFET5
Connections:
- Alert pad 1: Net-(AlertLED1-Pad1) -> Net-(AlertLED1-K)
- Alert pad 2: /LEDOUT -> Net-(AlertLED1-A)
- C1 pad 2: GNDREF -> GND
- C2 pad 2: GNDREF -> GND
- C3 pad 2: GNDREF -> GND
- C4 pad 2: GNDREF -> GND
- C5 pad 1: GNDREF -> GND
- R1 pad 2: GNDREF -> GND
- R2 pad 2: GNDREF -> GND
- R3 pad 2: GNDREF -> GND
- R4 pad 2: GNDREF -> GND
- R5 pad 2: GNDREF -> GND
- R8 pad 1: /LEDOUT -> Net-(AlertLED1-K)
- R8 pad 2: GNDREF -> GND
- U1 pad 11: /AS0 -> GND
- U1 pad 12: Net-(AlertLED1-Pad1) -> Net-(AlertLED1-A)
- U1 pad 13: /AS1 -> GND
- U1 pad 17: unconnected-(U1-Pad17) -> +3V3
- U1 pad 18: GNDREF -> GND
- U1 pad 21: GNDREF -> GND
- U1 pad 4: GNDREF -> GND
- U1 pad 5: GNDREF -> GND
- U1 pad 6: GNDREF -> GND
- U1 pad 9: GNDREF -> GND
Routing:
- net GNDREF: track 100.1 -> 0.00 mm, vias 14 -> 0
- net /AS0: track 48.1 -> 0.00 mm
- net /AS1: track 46.2 -> 0.00 mm
- net +3V3: track 80.5 -> 51.3 mm, vias 1 -> 5
- net /LEDOUT: track 22.1 -> 0.00 mm, vias 2 -> 0
- net Net-(AlertLED1-Pad1): track 13.8 -> 0.00 mm, vias 2 -> 0
- net Net-(U1-DCAP): track 10.4 -> 2.51 mm
- net /V_ref: track 55.8 -> 63.2 mm, vias 2 -> 0
- net /Vin2: track 19.3 -> 13.9 mm, vias 2 -> 0
- net /Vin4: track 17.2 -> 22.4 mm, vias 2 -> 0
- net Net-(AlertLED1-A): track 0.00 -> 2.98 mm
- net /Vin3: track 14.8 -> 17.0 mm
- net Net-(AlertLED1-K): track 0.00 -> 1.60 mm
- net /Vin5: track 27.9 -> 28.4 mm, vias 2 -> 0
- net /SCL_chip: track 62.5 -> 62.6 mm, vias 2 -> 0
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- added copper zone on B.Cu, net GND
- added copper zone on F.Cu, net GND
- removed copper zone on B.Cu, net GNDREF
Other:
- board size 92.9 x 34.7 mm -> 92.8 x 32.5 mm
