File: SunSensor/SunSensor.kicad_sch (KiCad schematic)
At the start: 16 parts, among them U1 AD7291BCPZ

Commit message: fixing kicad-libs
Parts:
- AlertLED1: footprint Display:HDSP-4836 -> sunsensor:LED_77&slash_TR8_EVE
- C1: footprint (none) -> sunsensor:CAPC1005X60N
- C2: footprint (none) -> sunsensor:CAPC3216X190N
- C3: footprint (none) -> sunsensor:CAPC1005X55N
- R10, R2, R4, R6, R8: footprint (none) -> sunsensor:RESC3116X65N
- R11: footprint (none) -> sunsensor:RESC3216X75N
- U1: footprint (none) -> sunsensor:QFN50P400X400X100-21N
- gave numbers to parts that had none: 5
Changed lines of the file:
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@@
       (effects (font (size 1 1) bold italic))
     )
-    (property "Footprint" "" (id 2) (at 105.41 35.56 0)
+    (property "Footprint" "sunsensor:QFN50P400X400X100-21N" (id 2) (at 105.41 35.56 0)
       (effects (font (size 1.27 1.27)) hide)
     )
@@
       (effects (font (size 1.27 1.27)) (justify left))
     )
-    (property "Footprint" "" (id 2) (at 110.1852 78.74 0)
+    (property "Footprint" "sunsensor:CAPC1005X60N" (id 2) (at 110.1852 78.74 0)
       (effects (font (size 1.27 1.27)) hide)
     )
@@
   (symbol (lib_id "4xxx:ALS-PT19-315C_L177_TR8") (at 60.96 21.59 0) (unit 1)
     (in_bom yes) (on_board yes)
-    (property "Reference" "MOSFET?" (id 0) (at 63.5 25.4 0)
+    (property "Reference" "MOSFET5" (id 0) (at 63.5 25.4 0)
       (effects (font (size 1.524 1.524)) (justify left))
     )
@@
       (effects (font (size 1.524 1.524)) (justify left))
     )
-    (property "Footprint" "sunsensor:LED_77&slash_TR8_EVE" (id 2) (at 60.96 21.59 0)
-      (effects (font (size 1.27 1.27) italic) hide)
+    (property "Footprint" "sunsensor:LED_77&slash_TR8_EVE" (id 2) (at 57.15 19.05 0)
+      (effects (font (size 1.27 1.27) italic))
     )
     (property "Datasheet" "ALS-PT19-315C/L177/TR8" (id 3) (at 60.96 21.59 0)
@@
   (symbol (lib_id "4xxx:ALS-PT19-315C_L177_TR8") (at 24.13 57.15 0) (unit 1)
     (in_bom yes) (on_board yes)
-    (property "Reference" "MOSFET?" (id 0) (at 26.67 60.96 0)
+    (property "Reference" "MOSFET2" (id 0) (at 26.67 60.96 0)
       (effects (font (size 1.524 1.524)) (justify left))
     )
@@
       (effects (font (size 1.27 1.27)) (justify left))
     )
-    (property "Footprint" "" (id 2) (at 43.18 74.93 0)
+    (property "Footprint" "sunsensor:RESC3116X65N" (id 2) (at 43.18 74.93 0)
       (effects (font (size 1.27 1.27)) hide)
     )
@@
   (symbol (lib_id "4xxx:ALS-PT19-315C_L177_TR8") (at 43.18 57.15 0) (unit 1)
     (in_bom yes) (on_board yes)
-    (property "Reference" "MOSFET?" (id 0) (at 45.72 60.96 0)
+    (property "Reference" "MOSFET4" (id 0) (at 45.72 60.96 0)
       (effects (font (size 1.524 1.524)) (justify left))
     )
@@
       (effects (font (size 1.27 1.27)) (justify left))
     )
-    (property "Footprint" "" (id 2) (at 133.0452 81.28 0)
+    (property "Footprint" "sunsensor:CAPC3216X190N" (id 2) (at 133.0452 81.28 0)
       (effects (font (size 1.27 1.27)) hide)
     )
@@
       (effects (font (size 1.27 1.27)) (justify left))
     )
-    (property "Footprint" "" (id 2) (at 60.96 40.64 0)
+    (property "Footprint" "sunsensor:RESC3116X65N" (id 2) (at 60.96 40.64 0)
       (effects (font (size 1.27 1.27)) hide)
     )
@@
   (symbol (lib_id "4xxx:ALS-PT19-315C_L177_TR8") (at 39.37 22.86 0) (unit 1)
     (in_bom yes) (on_board yes)
-    (property "Reference" "MOSFET?" (id 0) (at 41.91 26.67 0)
+    (property "Reference" "MOSFET3" (id 0) (at 41.91 26.67 0)
       (effects (font (size 1.524 1.524)) (justify left))
     )
@@
     (property "Reference" "AlertLED1" (id 0) (at 140.97 44.45 0))
     (property "Value" " " (id 1) (at 140.97 45.72 0))
-    (property "Footprint" "Display:HDSP-4836" (id 2) (at 140.97 57.15 0)
+    (property "Footprint" "sunsensor:LED_77&slash_TR8_EVE" (id 2) (at 140.97 57.15 0)
       (effects (font (size 1.27 1.27)) hide)
     )
@@
       (effects (font (size 1.27 1.27)) (justify left))
     )
-    (property "Footprint" "" (id 2) (at 24.13 74.93 0)
+    (property "Footprint" "sunsensor:RESC3116X65N" (id 2) (at 24.13 74.93 0)
       (effects (font (size 1.27 1.27)) hide)
     )
@@
     (property "Reference" "R11" (id 0) (at 153.67 43.18 90))
     (property "Value" "1k_ohms" (id 1) (at 153.67 45.72 90))
-    (property "Footprint" "" (id 2) (at 153.67 49.53 0)
+    (property "Footprint" "sunsensor:RESC3216X75N" (id 2) (at 153.67 49.53 0)
       (effects (font (size 1.27 1.27)) hide)
     )
@@
       (effects (font (size 1.27 1.27)) (justify left))
     )
-    (property "Footprint" "" (id 2) (at 39.37 40.64 0)
+    (property "Footprint" "sunsensor:RESC3116X65N" (id 2) (at 39.37 40.64 0)
       (effects (font (size 1.27 1.27)) hide)
     )
@@
       (effects (font (size 1.27 1.27)) (justify left))
     )
-    (property "Footprint" "" (id 2) (at 19.05 40.64 0)
+    (property "Footprint" "sunsensor:RESC3116X65N" (id 2) (at 19.05 40.64 0)
       (effects (font (size 1.27 1.27)) hide)
     )
@@
       (effects (font (size 1.27 1.27)) (justify left))
     )
-    (property "Footprint" "" (id 2) (at 147.0152 81.28 0)
+    (property "Footprint" "sunsensor:CAPC1005X55N" (id 2) (at 147.0152 81.28 0)
       (effects (font (size 1.27 1.27)) hide)
     )
@@
   (symbol (lib_id "4xxx:ALS-PT19-315C_L177_TR8") (at 19.05 22.86 0) (unit 1)
     (in_bom yes) (on_board yes)
-    (property "Reference" "MOSFET?" (id 0) (at 21.59 26.67 0)
+    (property "Reference" "MOSFET1" (id 0) (at 21.59 26.67 0)
       (effects (font (size 1.524 1.524)) (justify left))
     )
@@
     )
     (path "/ad949c33-8432-49a9-bb70-f0f6df65880e"
-      (reference "AlertLED1") (unit 1) (value " ") (footprint "Display:HDSP-4836")
+      (reference "AlertLED1") (unit 1) (value " ") (footprint "sunsensor:LED_77&slash_TR8_EVE")
     )
     (path "/390c528d-30f9-45ab-9bc5-65cc46896c9e"
-      (reference "C1") (unit 1) (value "1 µF") (footprint "")
+      (reference "C1") (unit 1) (value "1 µF") (footprint "sunsensor:CAPC1005X60N")
     )
     (path "/6b40ad9b-a415-46d0-a0b1-745e488e627b"
-      (reference "C2") (unit 1) (value "100 µF") (footprint "")
+      (reference "C2") (unit 1) (value "100 µF") (footprint "sunsensor:CAPC3216X190N")
     )
     (path "/f37a2f00-86ac-452a-9880-a4f0824a6e8b"
-      (reference "C3") (unit 1) (value "100 nF") (footprint "")
+      (reference "C3") (unit 1) (value "100 nF") (footprint "sunsensor:CAPC1005X55N")
+    )
+    (path "/f5ee5bf9-7b96-422f-bc88-1073f9c6dd48"
+      (reference "MOSFET1") (unit 1) (value "ALS-PT19") (footprint "sunsensor:LED_77&slash_TR8_EVE")
+    )
+    (path "/3e82bc40-c7e4-4bca-adb7-6ae68f4009fd"
+      (reference "MOSFET2") (unit 1) (value "ALS-PT19") (footprint "sunsensor:LED_77&slash_TR8_EVE")
+    )
+    (path "/9d4f76fb-88b0-4f7b-8c82-1de5c5eb9a9b"
+      (reference "MOSFET3") (unit 1) (value "ALS-PT19") (footprint "sunsensor:LED_77&slash_TR8_EVE")
+    )
+    (path "/69b5961c-3bef-402d-a9ec-105663dbf10e"
+      (reference "MOSFET4") (unit 1) (value "ALS-PT19") (footprint "sunsensor:LED_77&slash_TR8_EVE")
     )
     (path "/3b5f025d-15cd-40dc-91e1-f60e72eeda01"
-      (reference "MOSFET?") (unit 1) (value "ALS-PT19") (footprint "sunsensor:LED_77&slash_TR8_EVE")
-    )
-    (path "/3e82bc40-c7e4-4bca-adb7-6ae68f4009fd"
-      (reference "MOSFET?") (unit 1) (value "ALS-PT19") (footprint "sunsensor:LED_77&slash_TR8_EVE")
-    )
-    (path "/69b5961c-3bef-402d-a9ec-105663dbf10e"
-      (reference "MOSFET?") (unit 1) (value "ALS-PT19") (footprint "sunsensor:LED_77&slash_TR8_EVE")
-    )
-    (path "/9d4f76fb-88b0-4f7b-8c82-1de5c5eb9a9b"
-      (reference "MOSFET?") (unit 1) (value "ALS-PT19") (footprint "sunsensor:LED_77&slash_TR8_EVE")
-    )
-    (path "/f5ee5bf9-7b96-422f-bc88-1073f9c6dd48"
-      (reference "MOSFET?") (unit 1) (value "ALS-PT19") (footprint "sunsensor:LED_77&slash_TR8_EVE")
+      (reference "MOSFET5") (unit 1) (value "ALS-PT19") (footprint "sunsensor:LED_77&slash_TR8_EVE")
     )
     (path "/e8817e8b-6060-408d-9871-2edf3ddb6382"
-      (reference "R2") (unit 1) (value "50k_Ohms") (footprint "")
+      (reference "R2") (unit 1) (value "50k_Ohms") (footprint "sunsensor:RESC3116X65N")
     )
     (path "/afce43fa-2fc0-4ec3-8439-5ae0b899c7a3"
-      (reference "R4") (unit 1) (value "50k_Ohms") (footprint "")
+      (reference "R4") (unit 1) (value "50k_Ohms") (footprint "sunsensor:RESC3116X65N")
     )
     (path "/cdbd5bb7-c5cb-4058-9402-4d030cd77c46"
-      (reference "R6") (unit 1) (value "50k_Ohms") (footprint "")
+      (reference "R6") (unit 1) (value "50k_Ohms") (footprint "sunsensor:RESC3116X65N")
     )
     (path "/45650ad9-560e-49ac-a909-aa1ef50dfbce"
-      (reference "R8") (unit 1) (value "50k_Ohms") (footprint "")
+      (reference "R8") (unit 1) (value "50k_Ohms") (footprint "sunsensor:RESC3116X65N")
     )
     (path "/8f46fb76-00b9-4ac7-be29-c63d0348e4e9"
-      (reference "R10") (unit 1) (value "50k_Ohms") (footprint "")
+      (reference "R10") (unit 1) (value "50k_Ohms") (footprint "sunsensor:RESC3116X65N")
     )
     (path "/c262b603-0bd7-4242-a67f-7dedca9d95d6"
-      (reference "R11") (unit 1) (value "1k_ohms") (footprint "")
+      (reference "R11") (unit 1) (value "1k_ohms") (footprint "sunsensor:RESC3216X75N")
     )
     (path "/1c9b41c8-3f30-4b18-813d-639c8926d02e"
-      (reference "U1") (unit 1) (value "AD7291BCPZ") (footprint "")
-    )
-  )
+      (reference "U1") (unit 1) (value "AD7291BCPZ") (footprint "sunsensor:QFN50P400X400X100-21N")
+    )
+  )

Commit message: Finished traces
Parts:
- added U2: FEATHER_M0_BASIC_PROTO, MODULE_FEATHER_M0_BASIC_PROTO, symbol sunsensor:FEATHER_M0_BASIC_PROTO
Connections:
- net +3V3: now also U1.16 (VDRIVE), U2.P1_15 (3V3)
- net GNDREF: now also C1.2, C2.2, C3.2, U2.P1_1 (GND), U2.P1_13 (GND)
- net GNDS: no longer C1.2, C2.2, C3.2
- net AS0: now reaches U1.11 (AS0)
- net AS0: now also U2.P2_5 (PA19/EINT/I2SD0)
- net AS1: now reaches U1.13 (AS1)
- net AS1: now also U2.P2_4 (PA17/EINT/I2C)
- net SDA_chip: now reaches U1.14 (SDA)
- net SDA_chip: now also U2.P2_12 (PA22/EINT/I2C/SDA)
- net SCL_chip: now reaches U1.15 (SCL)
- net SCL_chip: now also U2.P2_11 (PA23/EINT/I2C/SCL)
Other:
- note added: "Signal Ground and Regular Ground or filter circuit? Separate Grounding planes"

Commit message: Final modifications
Parts:
- added C4: 10 µF, sunsensor:CAPC1005X71N, symbol Device:C
Connections:
- net GNDS: now also C4.2
- net V_ref: now also C4.1
- net LEDOUT: now reaches AlertLED1.20 (K), R11.1
Other:
- note removed: "Signal Ground and Regular Ground or filter circuit? Separate Grounding planes"
- moved on the sheet: R11
Changed lines of the file:
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@@
     (stroke (width 0) (type default) (color 0 0 0 0))
   )
-  (wire (pts (xy 161.29 49.53) (xy 161.29 52.07))
+  (wire (pts (xy 167.64 64.77) (xy 168.91 64.77))
     (stroke (width 0) (type default) (color 0 0 0 0))
   )
@@
     (stroke (width 0) (type default) (color 0 0 0 0))
   )
-  (wire (pts (xy 146.05 49.53) (xy 151.13 49.53))
-    (stroke (width 0) (type default) (color 0 0 0 0))
-  )
   (wire (pts (xy 24.13 67.31) (xy 24.13 69.85))
     (stroke (width 0) (type default) (color 0 0 0 0))
@@
     (stroke (width 0) (type default) (color 0 0 0 0))
   )
-  (wire (pts (xy 105.41 59.69) (xy 105.41 64.77))
-    (stroke (width 0) (type default) (color 0 0 0 0))
-  )
   (wire (pts (xy 83.82 50.8) (xy 92.71 50.8))
     (stroke (width 0) (type default) (color 0 0 0 0))
@@
     (stroke (width 0) (type default) (color 0 0 0 0))
   )
-  (wire (pts (xy 156.21 49.53) (xy 161.29 49.53))
+  (wire (pts (xy 147.32 49.53) (xy 146.05 49.53))
     (stroke (width 0) (type default) (color 0 0 0 0))
   )
@@
     (stroke (width 0) (type default) (color 0 0 0 0))
   )
-  (text "Signal Ground and Regular Ground or filter circuit?\n\nSeparate Grounding planes\n"
-    (at 40.64 99.06 0)
-    (effects (font (size 1.27 1.27)) (justify left bottom))
+  (wire (pts (xy 105.41 59.69) (xy 105.41 66.04))
+    (stroke (width 0) (type default) (color 0 0 0 0))
   )
   (label "Vin4" (at 81.28 39.37 0)
@@
   (label "Vin5" (at 46.99 69.85 0)
     (effects (font (size 1.27 1.27)) (justify left bottom))
+  )
+  (label "LEDOUT" (at 162.56 64.77 180)
+    (effects (font (size 1.27 1.27)) (justify right bottom))
   )
   (label "Vin2" (at 44.45 35.56 0)
@@
   )
   (label "V_ref" (at 39.37 19.05 0)
+    (effects (font (size 1.27 1.27)) (justify left bottom))
+  )
+  (label "LEDOUT" (at 147.32 49.53 0)
     (effects (font (size 1.27 1.27)) (justify left bottom))
   )
@@
     (pin "1")
   )
+  (symbol (lib_id "Device:C") (at 105.41 69.85 0) (unit 1)
+    (in_bom yes) (on_board yes)
+    (property "Reference" "C4" (id 0) (at 95.25 69.85 0)
+      (effects (font (size 1.27 1.27)) (justify left))
+    )
+    (property "Value" "10 µF" (id 1) (at 95.25 72.39 0)
+      (effects (font (size 1.27 1.27)) (justify left))
+    )
+    (property "Footprint" "sunsensor:CAPC1005X71N" (id 2) (at 106.3752 73.66 0)
+      (effects (font (size 1.27 1.27)) hide)
+    )
+    (property "Datasheet" "~" (id 3) (at 105.41 69.85 0)
+      (effects (font (size 1.27 1.27)) hide)
+    )
+    (pin "1")
+    (pin "2")
+  )
   (symbol (lib_id "Device:C") (at 109.22 74.93 0) (unit 1)
     (in_bom yes) (on_board yes)
@@
     (pin "2")
   )
+  (symbol (lib_id "power:GNDS") (at 105.41 73.66 0) (unit 1)
+    (in_bom yes) (on_board yes) (fields_autoplaced)
+    (property "Reference" "#PWR0103" (id 0) (at 105.41 80.01 0)
+      (effects (font (size 1.27 1.27)) hide)
+    )
+    (property "Value" "GNDS" (id 1) (at 105.41 78.74 0))
+    (property "Footprint" "" (id 2) (at 105.41 73.66 0)
+      (effects (font (size 1.27 1.27)) hide)
+    )
+    (property "Datasheet" "" (id 3) (at 105.41 73.66 0)
+      (effects (font (size 1.27 1.27)) hide)
+    )
+    (pin "1")
+  )
   (symbol (lib_id "4xxx:ALS-PT19-315C_L177_TR8") (at 43.18 57.15 0) (unit 1)
     (in_bom yes) (on_board yes)
@@
     (pin "1")
   )
-  (symbol (lib_id "power:GNDREF") (at 161.29 52.07 0) (unit 1)
-    (in_bom yes) (on_board yes) (fields_autoplaced)
-    (property "Reference" "#PWR021" (id 0) (at 161.29 58.42 0)
-      (effects (font (size 1.27 1.27)) hide)
-    )
-    (property "Value" "GNDREF" (id 1) (at 161.29 57.15 0))
-    (property "Footprint" "" (id 2) (at 161.29 52.07 0)
-      (effects (font (size 1.27 1.27)) hide)
-    )
-    (property "Datasheet" "" (id 3) (at 161.29 52.07 0)
+  (symbol (lib_id "power:GNDREF") (at 168.91 64.77 90) (unit 1)
+    (in_bom yes) (on_board yes) (fields_autoplaced)
+    (property "Reference" "#PWR021" (id 0) (at 175.26 64.77 0)
+      (effects (font (size 1.27 1.27)) hide)
+    )
+    (property "Value" "GNDREF" (id 1) (at 172.72 64.7699 90)
+      (effects (font (size 1.27 1.27)) (justify right))
+    )
+    (property "Footprint" "" (id 2) (at 168.91 64.77 0)
+      (effects (font (size 1.27 1.27)) hide)
+    )
+    (property "Datasheet" "" (id 3) (at 168.91 64.77 0)
       (effects (font (size 1.27 1.27)) hide)
     )
@@
     (pin "1")
   )
-  (symbol (lib_id "Device:50k_Ohms") (at 153.67 49.53 90) (unit 1)
-    (in_bom yes) (on_board yes) (fields_autoplaced)
-    (property "Reference" "R11" (id 0) (at 153.67 43.18 90))
-    (property "Value" "1k_ohms" (id 1) (at 153.67 45.72 90))
-    (property "Footprint" "sunsensor:RESC3216X75N" (id 2) (at 153.67 49.53 0)
-      (effects (font (size 1.27 1.27)) hide)
-    )
-    (property "Datasheet" "~" (id 3) (at 153.67 49.53 0)
+  (symbol (lib_id "Device:50k_Ohms") (at 165.1 64.77 90) (unit 1)
+    (in_bom yes) (on_board yes) (fields_autoplaced)
+    (property "Reference" "R11" (id 0) (at 165.1 58.42 90))
+    (property "Value" "1k_ohms" (id 1) (at 165.1 60.96 90))
+    (property "Footprint" "sunsensor:RESC3216X75N" (id 2) (at 165.1 64.77 0)
+      (effects (font (size 1.27 1.27)) hide)
+    )
+    (property "Datasheet" "~" (id 3) (at 165.1 64.77 0)
       (effects (font (size 1.27 1.27)) hide)
     )
@@
       (reference "#PWR0102") (unit 1) (value "GNDREF") (footprint "")
     )
+    (path "/689b33c2-41f4-422c-869a-3b64a4dff4d5"
+      (reference "#PWR0103") (unit 1) (value "GNDS") (footprint "")
+    )
     (path "/ad949c33-8432-49a9-bb70-f0f6df65880e"
       (reference "AlertLED1") (unit 1) (value " ") (footprint "sunsensor:LED_77&slash_TR8_EVE")
@@
       (reference "C3") (unit 1) (value "100 nF") (footprint "sunsensor:CAPC1005X55N")
     )
+    (path "/368ffb86-ddc0-4f87-80f0-47a79df5bd64"
+      (reference "C4") (unit 1) (value "10 µF") (footprint "sunsensor:CAPC1005X71N")
+    )
     (path "/f5ee5bf9-7b96-422f-bc88-1073f9c6dd48"

Commit message: Small fixes
Parts:
- added C5: 10 µF, sunsensor:CAPC1005X71N, symbol Device:C
Connections:
- net +3V3: now also C5.2
- net GNDS: now also C5.1
Changed lines of the file:
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@@
   (junction (at 19.05 35.56) (diameter 0) (color 0 0 0 0)
   )
+  (junction (at 121.92 21.59) (diameter 0) (color 0 0 0 0)
+  )
   (wire (pts (xy 39.37 35.56) (xy 39.37 38.1))
     (stroke (width 0) (type default) (color 0 0 0 0))
@@
     (stroke (width 0) (type default) (color 0 0 0 0))
   )
+  (wire (pts (xy 121.92 21.59) (xy 127 21.59))
+    (stroke (width 0) (type default) (color 0 0 0 0))
+  )
   (wire (pts (xy 254 76.2) (xy 254 80.01))
     (stroke (width 0) (type default) (color 0 0 0 0))
@@
     (stroke (width 0) (type default) (color 0 0 0 0))
   )
-  (wire (pts (xy 118.11 21.59) (xy 127 21.59))
+  (wire (pts (xy 118.11 21.59) (xy 121.92 21.59))
     (stroke (width 0) (type default) (color 0 0 0 0))
   )
@@
     (pin "9")
   )
+  (symbol (lib_id "Device:C") (at 121.92 17.78 0) (unit 1)
+    (in_bom yes) (on_board yes)
+    (property "Reference" "C5" (id 0) (at 111.76 17.78 0)
+      (effects (font (size 1.27 1.27)) (justify left))
+    )
+    (property "Value" "10 µF" (id 1) (at 111.76 20.32 0)
+      (effects (font (size 1.27 1.27)) (justify left))
+    )
+    (property "Footprint" "sunsensor:CAPC1005X71N" (id 2) (at 122.8852 21.59 0)
+      (effects (font (size 1.27 1.27)) hide)
+    )
+    (property "Datasheet" "~" (id 3) (at 121.92 17.78 0)
+      (effects (font (size 1.27 1.27)) hide)
+    )
+    (pin "1")
+    (pin "2")
+  )
   (symbol (lib_id "power:GNDREF") (at 39.37 43.18 0) (unit 1)
     (in_bom yes) (on_board yes) (fields_autoplaced)
@@
     (pin "1")
     (pin "2")
+  )
+  (symbol (lib_id "power:GNDS") (at 121.92 13.97 270) (unit 1)
+    (in_bom yes) (on_board yes) (fields_autoplaced)
+    (property "Reference" "#PWR0104" (id 0) (at 115.57 13.97 0)
+      (effects (font (size 1.27 1.27)) hide)
+    )
+    (property "Value" "GNDS" (id 1) (at 123.19 13.9699 90)
+      (effects (font (size 1.27 1.27)) (justify left))
+    )
+    (property "Footprint" "" (id 2) (at 121.92 13.97 0)
+      (effects (font (size 1.27 1.27)) hide)
+    )
+    (property "Datasheet" "" (id 3) (at 121.92 13.97 0)
+      (effects (font (size 1.27 1.27)) hide)
+    )
+    (pin "1")
   )
   (symbol (lib_id "LED:HDSP-4836") (at 140.97 49.53 0) (unit 1)
@@
       (reference "#PWR0103") (unit 1) (value "GNDS") (footprint "")
     )
+    (path "/a59acc7b-9355-407a-b9fc-642d4de9b341"
+      (reference "#PWR0104") (unit 1) (value "GNDS") (footprint "")
+    )
     (path "/ad949c33-8432-49a9-bb70-f0f6df65880e"
       (reference "AlertLED1") (unit 1) (value " ") (footprint "sunsensor:LED_77&slash_TR8_EVE")
@@
       (reference "C4") (unit 1) (value "10 µF") (footprint "sunsensor:CAPC1005X71N")
     )
+    (path "/26210416-31fe-4dd3-8d4c-c9168dffd369"
+      (reference "C5") (unit 1) (value "10 µF") (footprint "sunsensor:CAPC1005X71N")
+    )
     (path "/f5ee5bf9-7b96-422f-bc88-1073f9c6dd48"

Commit message: Finish Routing
Parts:
- added R6, R7: 10K, Resistor_SMD:R_0603_1608Metric, symbol Device:R_Small_US
- AlertLED1: footprint sunsensor:LED_77&slash_TR8_EVE -> LED_SMD:LED_0603_1608Metric; symbol LED:HDSP-4836 -> Device:LED
- C1: value 1 µF -> 1uF; footprint sunsensor:CAPC1005X60N -> Capacitor_SMD:C_0603_1608Metric
- C2: value 100 µF -> 10uF; footprint sunsensor:CAPC3216X190N -> Capacitor_SMD:C_0603_1608Metric
- C3: value 100 nF -> 0.1uF; footprint sunsensor:CAPC1005X55N -> Capacitor_SMD:C_0603_1608Metric
- C4: value 10 µF -> 10uF; footprint sunsensor:CAPC1005X71N -> Capacitor_SMD:C_0603_1608Metric
- C5: value 10 µF -> 1uF; footprint sunsensor:CAPC1005X71N -> Capacitor_SMD:C_0603_1608Metric
- MOSFET1: symbol 4xxx:ALS-PT19-315C_L177_TR8 -> SunSensor:ALS-PT19
- MOSFET2: renamed from MOSFET3; symbol 4xxx:ALS-PT19-315C_L177_TR8 -> SunSensor:ALS-PT19
- MOSFET3: renamed from MOSFET5; symbol 4xxx:ALS-PT19-315C_L177_TR8 -> SunSensor:ALS-PT19
- MOSFET4: renamed from MOSFET2; symbol 4xxx:ALS-PT19-315C_L177_TR8 -> SunSensor:ALS-PT19
- MOSFET5: renamed from MOSFET4; symbol 4xxx:ALS-PT19-315C_L177_TR8 -> SunSensor:ALS-PT19
- R1: renamed from R2; value 50k_Ohms -> 50K; footprint sunsensor:RESC3116X65N -> Resistor_SMD:R_0603_1608Metric; symbol Device:50k_Ohms -> Device:R_Small_US
- R2: renamed from R6; value 50k_Ohms -> 50K; footprint sunsensor:RESC3116X65N -> Resistor_SMD:R_0603_1608Metric; symbol Device:50k_Ohms -> Device:R_Small_US
- R3: renamed from R10; value 50k_Ohms -> 50K; footprint sunsensor:RESC3116X65N -> Resistor_SMD:R_0603_1608Metric; symbol Device:50k_Ohms -> Device:R_Small_US
- R4: value 50k_Ohms -> 50K; footprint sunsensor:RESC3116X65N -> Resistor_SMD:R_0603_1608Metric; symbol Device:50k_Ohms -> Device:R_Small_US
- R5: renamed from R8; value 50k_Ohms -> 50K; footprint sunsensor:RESC3116X65N -> Resistor_SMD:R_0603_1608Metric; symbol Device:50k_Ohms -> Device:R_Small_US
- R8: renamed from R11; value 1k_ohms -> 1K; footprint sunsensor:RESC3216X75N -> Resistor_SMD:R_0603_1608Metric; symbol Device:50k_Ohms -> Device:R_Small_US
- U1: footprint sunsensor:QFN50P400X400X100-21N -> Package_DFN_QFN:QFN-20-1EP_4x4mm_P0.5mm_EP2.6x2.6mm; symbol Analog_ADC:AD7291BCPZ -> SunSensor:AD7291BCPZ
- U2: footprint MODULE_FEATHER_M0_BASIC_PROTO -> Module:Adafruit_Feather; symbol sunsensor:FEATHER_M0_BASIC_PROTO -> MCU_Module:Adafruit_Feather_M0_Basic_Proto
Connections:
- net GNDS is gone; now on net GND: C4.2, C5.1, U1.18 (VIN0), U1.4 (VIN6), U1.5 (VIN7), U1.6 (GND1)
- net +3V3: now also U1.17 (PD/RST), U2.2 (3V3), R6.2, R7.2; no longer U2.P1_15 (3V3)
- net SCL_chip: now also U2.18 (SCL/D21), R6.1; no longer U2.P2_11 (PA23/EINT/I2C/SCL)
- net SDA_chip: now also U2.17 (SDA/D20), R7.1; no longer U2.P2_12 (PA22/EINT/I2C/SDA)
- net at U1.12 (Alert): now also AlertLED1.2 (A); no longer AlertLED1.1 (A)
- net AS0 renamed GND
- net GND: now also C1.2, C2.2, C3.2, R1.2, R2.2, R3.2, R4.2, R5.2, R8.2, U1.13 (AS1), U1.21 (GND), U1.9 (GND), U2.16 (GND), U2.4 (GND); no longer U2.P2_5 (PA19/EINT/I2SD0)
- removed net AS1: U1.13 (AS1), U2.P2_4 (PA17/EINT/I2C)
- removed net GNDREF: C1.2, C2.2, C3.2, R1.2, R2.2, R3.2, R4.2, R5.2, R8.2, U1.9 (GND), U2.P1_1 (GND), U2.P1_13 (GND)
- net LEDOUT: no longer names the net of R8.1
- net LEDOUT: now also AlertLED1.1 (K); no longer AlertLED1.20 (K)
- no-connect marks 0 -> 23
Other:
- moved on the sheet: AlertLED1, C1, C2, C3, C5, MOSFET1, MOSFET2, MOSFET3, MOSFET4, MOSFET5, R1, R2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
