File: SunSensorMux/SunSensorMux.kicad_sch (KiCad schematic)
At the start: 8 parts, among them J1 Conn_01x03, J2 Conn_01x03, U1 TCA9548A_Multiplexer

Commit message: fixing kicad-libs
Parts:
- L1, L2, L3, L4, L5: footprint (none) -> sunsensor:VEML7700-TR
Connections:
- net GND: no longer U1.20 (SCL7)
Changed lines of the file:
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@@
-    (pin "1")
-  )
-  (symbol (lib_id "power:GND") (at 90.17 121.92 90) (unit 1)
-    (in_bom yes) (on_board yes) (fields_autoplaced)
-    (property "Reference" "#PWR0117" (id 0) (at 96.52 121.92 0)
-      (effects (font (size 1.27 1.27)) hide)
-    )
-    (property "Value" "GND" (id 1) (at 93.98 121.9199 90)
-      (effects (font (size 1.27 1.27)) (justify right))
-    )
-    (property "Footprint" "" (id 2) (at 90.17 121.92 0)
-      (effects (font (size 1.27 1.27)) hide)
-    )
-    (property "Datasheet" "" (id 3) (at 90.17 121.92 0)
-      (effects (font (size 1.27 1.27)) hide)
-    )
     (pin "1")
   )
@@
       (effects (font (size 1.27 1.27)) (justify right))
     )
-    (property "Footprint" "" (id 2) (at 204.47 152.4 0)
+    (property "Footprint" "sunsensor:VEML7700-TR" (id 2) (at 204.47 152.4 0)
       (effects (font (size 1.27 1.27)) hide)
     )
@@
       (effects (font (size 1.27 1.27)) (justify left))
     )
-    (property "Footprint" "" (id 2) (at 214.63 17.78 0)
-      (effects (font (size 1.27 1.27)) hide)
-    )
+    (property "Footprint" "sunsensor:VEML7700-TR" (id 2) (at 214.63 17.78 0))
     (property "Datasheet" "" (id 3) (at 214.63 17.78 0)
       (effects (font (size 1.27 1.27)) hide)
@@
     (property "Reference" "L3" (id 0) (at 170.18 22.86 0))
     (property "Value" "VEML7700_Lux_Sensor" (id 1) (at 168.91 17.78 0))
-    (property "Footprint" "" (id 2) (at 170.18 17.78 0)
-      (effects (font (size 1.27 1.27)) hide)
-    )
+    (property "Footprint" "sunsensor:VEML7700-TR" (id 2) (at 170.18 17.78 0))
     (property "Datasheet" "" (id 3) (at 170.18 17.78 0)
       (effects (font (size 1.27 1.27)) hide)
@@
       (effects (font (size 1.27 1.27)) (justify left))
     )
-    (property "Footprint" "" (id 2) (at 120.65 19.05 0)
-      (effects (font (size 1.27 1.27)) hide)
-    )
+    (property "Footprint" "sunsensor:VEML7700-TR" (id 2) (at 120.65 19.05 0))
     (property "Datasheet" "" (id 3) (at 120.65 19.05 0)
       (effects (font (size 1.27 1.27)) hide)
@@
       (effects (font (size 1.27 1.27)) (justify right))
     )
-    (property "Footprint" "" (id 2) (at 127 154.94 0)
+    (property "Footprint" "sunsensor:VEML7700-TR" (id 2) (at 127 154.94 0)
       (effects (font (size 1.27 1.27)) hide)
     )
@@
       (reference "#PWR0115") (unit 1) (value "GND") (footprint "")
     )
-    (path "/058ebdda-7277-4b18-933e-2d889dd2e4ab"
-      (reference "#PWR0117") (unit 1) (value "GND") (footprint "")
-    )
     (path "/7260268d-6fca-4357-9436-cc17031d64b3"
       (reference "#PWR0118") (unit 1) (value "GND") (footprint "")
@@
     )
     (path "/7b6eea8d-d802-469d-a284-aaa27effb2a9"
-      (reference "L1") (unit 1) (value "VEML7700_Lux_Sensor") (footprint "")
+      (reference "L1") (unit 1) (value "VEML7700_Lux_Sensor") (footprint "sunsensor:VEML7700-TR")
     )
     (path "/e3a1db09-036e-4e18-a1c7-272198f2b9a1"
-      (reference "L2") (unit 1) (value "VEML7700_Lux_Sensor") (footprint "")
+      (reference "L2") (unit 1) (value "VEML7700_Lux_Sensor") (footprint "sunsensor:VEML7700-TR")
     )
     (path "/3d713675-1ff5-4d3c-811d-1db9d6c548c6"
-      (reference "L3") (unit 1) (value "VEML7700_Lux_Sensor") (footprint "")
+      (reference "L3") (unit 1) (value "VEML7700_Lux_Sensor") (footprint "sunsensor:VEML7700-TR")
     )
     (path "/0a948857-9a00-4016-9ea2-d6a3ee282cff"
-      (reference "L4") (unit 1) (value "VEML7700_Lux_Sensor") (footprint "")
+      (reference "L4") (unit 1) (value "VEML7700_Lux_Sensor") (footprint "sunsensor:VEML7700-TR")
     )
     (path "/3a3e63ad-022b-49c3-9917-663995f5b6c1"
-      (reference "L5") (unit 1) (value "VEML7700_Lux_Sensor") (footprint "")
+      (reference "L5") (unit 1) (value "VEML7700_Lux_Sensor") (footprint "sunsensor:VEML7700-TR")
     )
     (path "/2efcfa5b-9d9a-45e0-ac3e-7b62fcbcda6b"

Commit message: finished board
Parts:
- removed J1, J2: Conn_01x03, symbol Connector_Generic:Conn_01x03
- added U2: FEATHER_M0_BASIC_PROTO, sunsensor:MODULE_FEATHER_M0_BASIC_PROTO, symbol sunsensor:FEATHER_M0_BASIC_PROTO
Connections:
- net +3.3VDAC is gone; now on net +3V3: L1.2 (Vin), L2.2 (Vin), L3.2 (Vin), L4.2 (Vin), L5.2 (Vin)
- net GND: now also U2.P1_1 (GND), U2.P1_13 (GND)
- net at L4.1 (SCL): now also U1.11 (SCL3); no longer U1.14 (SCL4)
- net at U1.13 (SDA4): now also L2.4 (SDA); no longer L4.5 (SDA)
- net A0: now reaches U1.1 (A0)
- net A0: now also U2.P2_6 (PA16/EINT/I2C)
- net at U1.10 (SDA3): now also L4.4 (SDA); no longer L2.5 (SDA)
- net at L2.1 (SCL): now also U1.14 (SCL4); no longer U1.11 (SCL3)
- net A1: now reaches U1.2 (A1)
- net A1: now also U2.P2_5 (PA19/EINT/I2SD0)
- net A2: now reaches U1.21 (A2)
- net A2: now also U2.P2_4 (PA17/EINT/I2C)
- net SCL: now reaches U1.22 (SCL)
- net SCL: now also U2.P2_11 (PA23/EINT/I2C/SCL)
- net SDA: now reaches U1.23 (SDA)
- net SDA: now also U2.P2_12 (PA22/EINT/I2C/SDA)
- net +3V3: now reaches U1.24 (VCC)
- net +3V3: now also U2.P1_15 (3V3)
- net RESET: now reaches U1.3 (RESET)
- net RESET: now also U2.P2_7 (PA18/EINT)
- net at U1.4 (SDA0): now also L1.4 (SDA); no longer L1.5 (SDA)
- net at U1.6 (SDA1): now also L3.4 (SDA); no longer L3.5 (SDA)
- net at U1.8 (SDA2): now also L5.1 (SCL); no longer L5.5 (SDA)
- net at U1.9 (SCL2): now also L5.4 (SDA); no longer L5.1 (SCL)
Other:
- moved on the sheet: L1, L3, L4, L5, U1

Commit message: Final modifications
Connections:
- net SCL3: now reaches L4.1 (SCL), U1.11 (SCL3)
- net SDA3: now reaches L4.4 (SDA), U1.10 (SDA3)
- net SDA4: now reaches L2.4 (SDA), U1.13 (SDA4)
- net SCL4: now reaches L2.1 (SCL), U1.14 (SCL4)
- net SDA0: now reaches L1.4 (SDA), U1.4 (SDA0)
- net SCL0: now reaches L1.1 (SCL), U1.5 (SCL0)
- net SDA1: now reaches L3.4 (SDA), U1.6 (SDA1)
- net SCL1: now reaches L3.1 (SCL), U1.7 (SCL1)
- net SDA2: now reaches L5.1 (SCL), U1.8 (SDA2)
- net SCL2: now reaches L5.4 (SDA), U1.9 (SCL2)
Changed lines of the file:
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@@
 (kicad_sch (version 20211123) (generator eeschema)
   (paper "A4")
+  (junction (at 104.14 30.48) (diameter 0) (color 0 0 0 0)
+  )
   (wire (pts (xy 57.15 63.5) (xy 60.96 63.5))
     (stroke (width 0) (type default) (color 0 0 0 0))
@@
     (stroke (width 0) (type default) (color 0 0 0 0))
   )
+  (wire (pts (xy 105.41 30.48) (xy 104.14 30.48))
+    (stroke (width 0) (type default) (color 0 0 0 0))
+  )
   (wire (pts (xy 93.98 41.91) (xy 104.14 41.91))
     (stroke (width 0) (type default) (color 0 0 0 0))
@@
     (effects (font (size 1.27 1.27)) (justify left bottom))
   )
+  (label "SDA1" (at 60.96 36.83 0)
+    (effects (font (size 1.27 1.27)) (justify left bottom))
+  )
   (label "A1" (at 21.59 49.53 0)
     (effects (font (size 1.27 1.27)) (justify left bottom))
   )
+  (label "SDA3" (at 67.31 62.23 0)
+    (effects (font (size 1.27 1.27)) (justify left bottom))
+  )
+  (label "SCL3" (at 58.42 57.15 0)
+    (effects (font (size 1.27 1.27)) (justify left bottom))
+  )
+  (label "SCL4" (at 66.04 66.04 0)
+    (effects (font (size 1.27 1.27)) (justify left bottom))
+  )
   (label "A2" (at 21.59 45.72 0)
     (effects (font (size 1.27 1.27)) (justify left bottom))
   )
+  (label "SDA4" (at 58.42 63.5 0)
+    (effects (font (size 1.27 1.27)) (justify left bottom))
+  )
   (label "A0" (at 21.59 53.34 0)
     (effects (font (size 1.27 1.27)) (justify left bottom))
@@
     (effects (font (size 1.27 1.27)) (justify left bottom))
   )
+  (label "SCL0" (at 59.69 19.05 0)
+    (effects (font (size 1.27 1.27)) (justify left bottom))
+  )
   (label "RESET" (at 210.82 110.49 0)
     (effects (font (size 1.27 1.27)) (justify left bottom))
@@
     (effects (font (size 1.27 1.27)) (justify left bottom))
   )
+  (label "SCL1" (at 59.69 39.37 0)
+    (effects (font (size 1.27 1.27)) (justify left bottom))
+  )
   (label "SCL" (at 22.86 31.75 0)
     (effects (font (size 1.27 1.27)) (justify left bottom))
   )
   (label "A0" (at 210.82 107.95 0)
+    (effects (font (size 1.27 1.27)) (justify left bottom))
+  )
+  (label "SDA0" (at 63.5 30.48 0)
+    (effects (font (size 1.27 1.27)) (justify left bottom))
+  )
+  (label "SDA2" (at 59.69 44.45 0)
+    (effects (font (size 1.27 1.27)) (justify left bottom))
+  )
+  (label "SCL2" (at 58.42 48.26 0)
     (effects (font (size 1.27 1.27)) (justify left bottom))
   )
@@
   )
   (symbol (lib_id "power:+3.3V") (at 104.14 59.69 90) (unit 1)
-    (in_bom yes) (on_board yes) (fields_autoplaced)
+    (in_bom yes) (on_board yes)
     (property "Reference" "#PWR0108" (id 0) (at 107.95 59.69 0)
       (effects (font (size 1.27 1.27)) hide)
     )
-    (property "Value" "+3.3V" (id 1) (at 105.41 59.6899 90)
+    (property "Value" "+3.3V" (id 1) (at 105.41 62.23 90)
       (effects (font (size 1.27 1.27)) (justify right))
     )
@@
   )
   (symbol (lib_id "power:+3.3V") (at 68.58 46.99 90) (unit 1)
-    (in_bom yes) (on_board yes) (fields_autoplaced)
+    (in_bom yes) (on_board yes)
     (property "Reference" "#PWR0101" (id 0) (at 72.39 46.99 0)
       (effects (font (size 1.27 1.27)) hide)
     )
-    (property "Value" "+3.3V" (id 1) (at 69.85 46.9899 90)
-      (effects (font (size 1.27 1.27)) (justify right))
-    )
+    (property "Value" "+3.3V" (id 1) (at 69.85 49.53 90)
+      (effects (font (size 1.27 1.27)) (justify right))
+    )

Commit message: Small fixes
Connections:
- net GND: now also U1.1 (A0), U1.2 (A1), U1.21 (A2)
- net SCL2: no longer L5.4 (SDA), U1.9 (SCL2)
- net SDA2: now also L5.4 (SDA); no longer L5.1 (SCL)
- net A0: no longer names the net of U2.P2_6 (PA16/EINT/I2C)
- net A0: no longer U1.1 (A0)
- net A1: no longer names the net of U2.P2_5 (PA19/EINT/I2SD0)
- net A1: no longer U1.2 (A1)
- net A2: no longer names the net of U2.P2_4 (PA17/EINT/I2C)
- net A2: no longer U1.21 (A2)
- new net: L5.1 (SCL), U1.9 (SCL2)
Changed lines of the file:
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@@
   (junction (at 104.14 30.48) (diameter 0) (color 0 0 0 0)
   )
+  (junction (at 21.59 49.53) (diameter 0) (color 0 0 0 0)
+  )
+  (junction (at 21.59 53.34) (diameter 0) (color 0 0 0 0)
+  )
   (wire (pts (xy 57.15 63.5) (xy 60.96 63.5))
     (stroke (width 0) (type default) (color 0 0 0 0))
@@
     (stroke (width 0) (type default) (color 0 0 0 0))
   )
+  (wire (pts (xy 64.77 46.99) (xy 64.77 44.45))
+    (stroke (width 0) (type default) (color 0 0 0 0))
+  )
   (wire (pts (xy 59.69 31.75) (xy 59.69 19.05))
     (stroke (width 0) (type default) (color 0 0 0 0))
   )
-  (wire (pts (xy 66.04 53.34) (xy 66.04 55.88))
-    (stroke (width 0) (type default) (color 0 0 0 0))
-  )
   (wire (pts (xy 104.14 38.1) (xy 101.6 38.1))
     (stroke (width 0) (type default) (color 0 0 0 0))
@@
     (stroke (width 0) (type default) (color 0 0 0 0))
   )
-  (wire (pts (xy 58.42 46.99) (xy 58.42 53.34))
-    (stroke (width 0) (type default) (color 0 0 0 0))
-  )
   (wire (pts (xy 105.41 30.48) (xy 104.14 30.48))
     (stroke (width 0) (type default) (color 0 0 0 0))
   )
+  (wire (pts (xy 57.15 44.45) (xy 63.5 44.45))
+    (stroke (width 0) (type default) (color 0 0 0 0))
+  )
   (wire (pts (xy 93.98 41.91) (xy 104.14 41.91))
     (stroke (width 0) (type default) (color 0 0 0 0))
@@
     (stroke (width 0) (type default) (color 0 0 0 0))
   )
-  (wire (pts (xy 57.15 44.45) (xy 68.58 44.45))
-    (stroke (width 0) (type default) (color 0 0 0 0))
-  )
-  (wire (pts (xy 66.04 55.88) (xy 68.58 55.88))
-    (stroke (width 0) (type default) (color 0 0 0 0))
-  )
   (wire (pts (xy 63.5 54.61) (xy 63.5 62.23))
     (stroke (width 0) (type default) (color 0 0 0 0))
@@
     (stroke (width 0) (type default) (color 0 0 0 0))
   )
+  (wire (pts (xy 21.59 53.34) (xy 21.59 57.15))
+    (stroke (width 0) (type default) (color 0 0 0 0))
+  )
   (wire (pts (xy 22.86 31.75) (xy 27.94 31.75))
     (stroke (width 0) (type default) (color 0 0 0 0))
@@
     (stroke (width 0) (type default) (color 0 0 0 0))
   )
-  (wire (pts (xy 58.42 53.34) (xy 66.04 53.34))
+  (wire (pts (xy 63.5 44.45) (xy 63.5 53.34))
     (stroke (width 0) (type default) (color 0 0 0 0))
   )
@@
     (stroke (width 0) (type default) (color 0 0 0 0))
   )
+  (wire (pts (xy 64.77 53.34) (xy 64.77 55.88))
+    (stroke (width 0) (type default) (color 0 0 0 0))
+  )
   (wire (pts (xy 93.98 36.83) (xy 93.98 41.91))
     (stroke (width 0) (type default) (color 0 0 0 0))
@@
     (stroke (width 0) (type default) (color 0 0 0 0))
   )
+  (wire (pts (xy 64.77 55.88) (xy 68.58 55.88))
+    (stroke (width 0) (type default) (color 0 0 0 0))
+  )
   (wire (pts (xy 63.5 29.21) (xy 63.5 30.48))
     (stroke (width 0) (type default) (color 0 0 0 0))
   )
+  (wire (pts (xy 64.77 44.45) (xy 68.58 44.45))
+    (stroke (width 0) (type default) (color 0 0 0 0))
+  )
+  (wire (pts (xy 21.59 45.72) (xy 21.59 49.53))
+    (stroke (width 0) (type default) (color 0 0 0 0))
+  )
   (wire (pts (xy 95.25 62.23) (xy 95.25 68.58))
     (stroke (width 0) (type default) (color 0 0 0 0))
@@
     (stroke (width 0) (type default) (color 0 0 0 0))
   )
+  (wire (pts (xy 63.5 53.34) (xy 64.77 53.34))
+    (stroke (width 0) (type default) (color 0 0 0 0))
+  )
   (wire (pts (xy 62.23 63.5) (xy 99.06 63.5))
     (stroke (width 0) (type default) (color 0 0 0 0))
@@
     (stroke (width 0) (type default) (color 0 0 0 0))
   )
-  (wire (pts (xy 57.15 46.99) (xy 58.42 46.99))
+  (wire (pts (xy 57.15 46.99) (xy 64.77 46.99))
+    (stroke (width 0) (type default) (color 0 0 0 0))
+  )
+  (wire (pts (xy 21.59 49.53) (xy 21.59 53.34))
     (stroke (width 0) (type default) (color 0 0 0 0))
   )
@@
     (effects (font (size 1.27 1.27)) (justify left bottom))
   )
-  (label "A1" (at 21.59 49.53 0)
-    (effects (font (size 1.27 1.27)) (justify left bottom))
-  )
   (label "SDA3" (at 67.31 62.23 0)
     (effects (font (size 1.27 1.27)) (justify left bottom))
@@
     (effects (font (size 1.27 1.27)) (justify left bottom))
   )
-  (label "A2" (at 21.59 45.72 0)
-    (effects (font (size 1.27 1.27)) (justify left bottom))
-  )
   (label "SDA4" (at 58.42 63.5 0)
     (effects (font (size 1.27 1.27)) (justify left bottom))
   )
-  (label "A0" (at 21.59 53.34 0)
-    (effects (font (size 1.27 1.27)) (justify left bottom))
-  )
   (label "RESET" (at 21.59 34.29 0)
     (effects (font (size 1.27 1.27)) (justify left bottom))
@@
     (effects (font (size 1.27 1.27)) (justify left bottom))
   )
-  (label "A2" (at 210.82 102.87 0)
-    (effects (font (size 1.27 1.27)) (justify left bottom))
-  )
   (label "SCL" (at 210.82 120.65 0)
     (effects (font (size 1.27 1.27)) (justify left bottom))
   )
-  (label "A1" (at 210.82 105.41 0)
-    (effects (font (size 1.27 1.27)) (justify left bottom))
-  )
   (label "SDA" (at 210.82 123.19 0)
     (effects (font (size 1.27 1.27)) (justify left bottom))
@@
   )
   (label "SCL" (at 22.86 31.75 0)
-    (effects (font (size 1.27 1.27)) (justify left bottom))
-  )
-  (label "A0" (at 210.82 107.95 0)
     (effects (font (size 1.27 1.27)) (justify left bottom))
   )
@@
     (pin "1")
   )
+  (symbol (lib_id "power:GND") (at 21.59 57.15 0) (unit 1)
+    (in_bom yes) (on_board yes) (fields_autoplaced)
+    (property "Reference" "#PWR0114" (id 0) (at 21.59 63.5 0)
+      (effects (font (size 1.27 1.27)) hide)
+    )
+    (property "Value" "GND" (id 1) (at 24.13 58.4199 0)
+      (effects (font (size 1.27 1.27)) (justify left))
+    )
+    (property "Footprint" "" (id 2) (at 21.59 57.15 0)
+      (effects (font (size 1.27 1.27)) hide)
+    )
+    (property "Datasheet" "" (id 3) (at 21.59 57.15 0)
+      (effects (font (size 1.27 1.27)) hide)
+    )
+    (pin "1")
+  )
   (symbol (lib_id "power:GND") (at 68.58 52.07 270) (unit 1)
     (in_bom yes) (on_board yes) (fields_autoplaced)
@@
       (reference "#PWR0113") (unit 1) (value "GND") (footprint "")
     )
+    (path "/af5998e9-d35a-4293-a024-885e8c412fce"
+      (reference "#PWR0114") (unit 1) (value "GND") (footprint "")
+    )
     (path "/b8f924c5-769f-47a5-afb6-d0c7ff32c076"

Commit message: Finish Routing
Parts:
- removed L2, L4, L5: VEML7700_Lux_Sensor, sunsensor:VEML7700-TR, symbol Sensor_Optical:VEML7700_Lux_Sensor
- added C1: 1uF, Capacitor_SMD:C_0603_1608Metric, symbol Device:C_Small
- added C2, C3, C4, C5, C6: 0.1uF, Capacitor_SMD:C_0603_1608Metric, symbol Device:C_Small
- added L2, L4, L5: VEML7700_Lux_Sensor, sunsensor:VEML7700-TT, symbol SunSensor:VEML7700_Lux_Sensor
- added R1, R10, R11, R12, R13, R2, R3, R4, R5, R6, R7, R8, R9: 10K, Resistor_SMD:R_0603_1608Metric, symbol Device:R_Small
- L1, L3: footprint sunsensor:VEML7700-TR -> sunsensor:VEML7700-TT; symbol Sensor_Optical:VEML7700_Lux_Sensor -> SunSensor:VEML7700_Lux_Sensor
- U1: footprint sunsensor:SOP65P640X120-24N -> Package_SO:TSSOP-24_4.4x7.8mm_P0.65mm; symbol Analog_Switch:TCA9548A_Multiplexer -> Interface_Expansion:TCA9548APWR
- U2: footprint sunsensor:MODULE_FEATHER_M0_BASIC_PROTO -> Module:Adafruit_Feather; symbol sunsensor:FEATHER_M0_BASIC_PROTO -> MCU_Module:Adafruit_Feather_M0_Basic_Proto
Connections:
- net GND: now also U2.16 (GND), U2.4 (GND), C1.2, C2.1, C3.1, C4.1, C5.1, C6.1, L2.3 (GND), L4.3 (GND), L5.3 (GND); no longer U1.15 (SDA5), U1.17 (SDA6), U1.19 (SDA7), U2.P1_1 (GND), U2.P1_13 (GND)
- net RESET: now also U2.19 (D5), R1.1; no longer U2.P2_7 (PA18/EINT)
- net SCL: now also U2.18 (SCL/D21), R3.1; no longer U2.P2_11 (PA23/EINT/I2C/SCL)
- net SCL0: now also R4.2
- net SCL1: now also L2.1 (SCL), R6.2; no longer L3.1 (SCL)
- net SCL2: now also L3.1 (SCL), U1.9 (SC2), R8.2
- net SCL3: now also L4.1 (SCL), R10.2
- net SCL4: now also L5.1 (SCL), R12.2
- net SDA: now also U2.17 (SDA/D20), R2.1; no longer U2.P2_12 (PA22/EINT/I2C/SDA)
- net SDA0: now also R5.2
- net SDA1: now also L2.4 (SDA), R7.2; no longer L3.4 (SDA)
- net SDA2: now also L3.4 (SDA), R9.2
- net SDA3: now also L4.4 (SDA), R11.2
- net SDA4: now also L5.4 (SDA), R13.2
- net SCL5: now reaches U1.16 (SC5)
- net SCL6: now reaches U1.18 (SC6)
- net SCL7: now reaches U1.20 (SC7)
- net +3V3 renamed +3.3V
- net +3.3V: now also U2.2 (3V3), C1.1, C2.2, C3.2, C4.2, C5.2, C6.2, L2.2 (Vin), L4.2 (Vin), L5.2 (Vin), R1.2, R10.1, R11.1, R12.1, R13.1, R2.2, R3.2, R4.1, R5.1, R6.1, R7.1, R8.1, R9.1; no longer U2.P1_15 (3V3)
- new net SDA5: U1.15 (SD5)
- new net SDA6: U1.17 (SD6)
- new net SDA7: U1.19 (SD7)
- no-connect marks 0 -> 22
Other:
- moved on the sheet: L1, L3
